Commit message: change gripper range and add mechanical parameters for the simulation

File: bme_ros_simple_arm/urdf/mogi_arm.xacro (robot description, xacro)
@@ -219,5 +219,5 @@
   <!-- Left finger joint -->
   <joint name="left_finger_joint" type="prismatic">
-    <limit lower="0" upper="0.03" effort="1000.0" velocity="4.0"/>
+    <limit lower="0" upper="0.04" effort="100.0" velocity="4.0"/>
     <parent link="gripper_base"/>
     <child link="left_finger"/>
@@ -250,13 +250,16 @@
   </link>
   <gazebo reference="left_finger">
-    <mu1>1.0</mu1>
-    <mu2>1.0</mu2>
-    <minDepth>0.003</minDepth>
-    <maxVel>0</maxVel>
+    <kp>1000000.0</kp>
+    <kd>100.0</kd>
+    <mu1>15</mu1>
+    <mu2>15</mu2>
+    <fdir1>1 0 0</fdir1>
+    <maxVel>1.0</maxVel>
+    <minDepth>0.002</minDepth>
     <material>Gazebo/Blue</material>
   </gazebo>
   <!-- Right finger joint -->
   <joint name="right_finger_joint" type="prismatic">
-    <limit lower="0" upper="0.03" effort="1000.0" velocity="4.0"/>
+    <limit lower="0" upper="0.04" effort="100.0" velocity="4.0"/>
     <parent link="gripper_base"/>
     <child link="right_finger"/>
@@ -289,8 +292,11 @@
   </link>
   <gazebo reference="right_finger">
-    <mu1>1.0</mu1>
-    <mu2>1.0</mu2>
-    <minDepth>0.003</minDepth>
-    <maxVel>0</maxVel>
+    <kp>1000000.0</kp>
+    <kd>100.0</kd>
+    <mu1>15</mu1>
+    <mu2>15</mu2>
+    <fdir1>1 0 0</fdir1>
+    <maxVel>1.0</maxVel>
+    <minDepth>0.002</minDepth>
     <material>Gazebo/Blue</material>
   </gazebo>

Commit message: add simulated gripper camera

File: bme_ros_simple_arm/urdf/mogi_arm.xacro (robot description, xacro)
@@ -324,3 +324,40 @@
     </inertial>
   </link>
+  <gazebo reference="end_effector_link">
+    <material>Gazebo/Red</material>
+  </gazebo>
+  <!-- Camera -->
+  <joint type="fixed" name="camera_joint">
+    <origin xyz="0.0 0.0 0.0" rpy="0 -1.5707 0"/>
+    <child link="camera_link"/>
+    <parent link="gripper_base"/>
+  </joint>
+  <link name='camera_link'>
+    <pose>0 0 0 0 0 0</pose>
+    <inertial>
+      <mass value="1.0e-03"/>
+      <origin xyz="0 0 0" rpy="0 0 0"/>
+      <inertia
+          ixx="1e-6" ixy="0" ixz="0"
+          iyy="1e-6" iyz="0"
+          izz="1e-6"
+      />
+    </inertial>
+    <visual name='camera_link_visual'>
+      <origin xyz="0 0 0" rpy="0 0 0"/>
+      <geometry>
+        <box size=".01 .01 .01"/>
+      </geometry>
+    </visual>
+  </link>
+  <gazebo reference="camera_link">
+    <material>Gazebo/Red</material>
+  </gazebo>
+  <joint type="fixed" name="camera_optical_joint">
+    <origin xyz="0 0 0" rpy="-1.5707 0 -1.5707"/>
+    <child link="camera_link_optical"/>
+    <parent link="camera_link"/>
+  </joint>
+  <link name="camera_link_optical">
+  </link>
 </robot>

Commit message: add a table camera

File: bme_ros_simple_arm/urdf/mogi_arm.xacro (robot description, xacro)
@@ -327,11 +327,11 @@
     <material>Gazebo/Red</material>
   </gazebo>
-  <!-- Camera -->
-  <joint type="fixed" name="camera_joint">
+  <!-- Gripper camera -->
+  <joint type="fixed" name="gripper_camera_joint">
     <origin xyz="0.0 0.0 0.0" rpy="0 -1.5707 0"/>
-    <child link="camera_link"/>
+    <child link="gripper_camera_link"/>
     <parent link="gripper_base"/>
   </joint>
-  <link name='camera_link'>
+  <link name='gripper_camera_link'>
     <pose>0 0 0 0 0 0</pose>
     <inertial>
@@ -344,5 +344,5 @@
       />
     </inertial>
-    <visual name='camera_link_visual'>
+    <visual>
       <origin xyz="0 0 0" rpy="0 0 0"/>
       <geometry>
@@ -351,13 +351,47 @@
     </visual>
   </link>
-  <gazebo reference="camera_link">
+  <gazebo reference="gripper_camera_link">
     <material>Gazebo/Red</material>
   </gazebo>
-  <joint type="fixed" name="camera_optical_joint">
+  <joint type="fixed" name="gripper_camera_optical_joint">
     <origin xyz="0 0 0" rpy="-1.5707 0 -1.5707"/>
-    <child link="camera_link_optical"/>
-    <parent link="camera_link"/>
-  </joint>
-  <link name="camera_link_optical">
+    <child link="gripper_camera_link_optical"/>
+    <parent link="gripper_camera_link"/>
+  </joint>
+  <link name="gripper_camera_link_optical">
+  </link>
+  <!-- Table camera -->
+  <joint type="fixed" name="table_camera_joint">
+    <origin xyz="1.0 0.4 0.2" rpy="0 0 3.6652"/>
+    <child link="table_camera_link"/>
+    <parent link="world"/>
+  </joint>
+  <link name='table_camera_link'>
+    <pose>0 0 0 0 0 0</pose>
+    <inertial>
+      <mass value="1.0e-03"/>
+      <origin xyz="0 0 0" rpy="0 0 0"/>
+      <inertia
+          ixx="1e-6" ixy="0" ixz="0"
+          iyy="1e-6" iyz="0"
+          izz="1e-6"
+      />
+    </inertial>
+    <visual>
+      <origin xyz="0 0 0" rpy="0 0 0"/>
+      <geometry>
+        <box size=".05 .05 .05"/>
+      </geometry>
+    </visual>
+  </link>
+  <gazebo reference="table_camera_link">
+    <material>Gazebo/Red</material>
+  </gazebo>
+  <joint type="fixed" name="table_camera_optical_joint">
+    <origin xyz="0 0 0" rpy="-1.5707 0 -1.5707"/>
+    <child link="table_camera_link_optical"/>
+    <parent link="table_camera_link"/>
+  </joint>
+  <link name="table_camera_link_optical">
   </link>
 </robot>

Commit message: add 3D models to URDF

File: bme_ros_simple_arm/urdf/mogi_arm.xacro (robot description, xacro)
@@ -67,5 +67,6 @@
     <visual>
       <geometry>
-        <cylinder radius="0.1" length="0.05"/>
+        <!--cylinder radius="0.1" length="0.05"/-->
+        <mesh filename = "package://bme_ros_simple_arm/meshes/shoulder.dae"/>
       </geometry>
       <material name="orange"/>
@@ -73,7 +74,7 @@
     </visual>
   </link>
-  <gazebo reference="shoulder_link">
+  <!--gazebo reference="shoulder_link">
     <material>Gazebo/Orange</material>
-  </gazebo>
+  </gazebo-->
   <!-- Shoulder lift joint -->
   <joint name="shoulder_lift_joint" type="revolute">
@@ -103,5 +104,6 @@
     <visual>
       <geometry>
-        <cylinder radius="0.05" length="0.2"/>
+        <!--cylinder radius="0.05" length="0.2"/-->
+        <mesh filename = "package://bme_ros_simple_arm/meshes/upper_arm.dae"/>
       </geometry>
       <material name="orange"/>
@@ -109,7 +111,7 @@
     </visual>
   </link>
-  <gazebo reference="upper_arm_link">
+  <!--gazebo reference="upper_arm_link">
     <material>Gazebo/Orange</material>
-  </gazebo>
+  </gazebo-->
   <!-- Elbow joint -->
   <joint name="elbow_joint" type="revolute">
@@ -139,5 +141,6 @@
     <visual>
       <geometry>
-        <cylinder radius="0.025" length="0.25"/>
+        <!--cylinder radius="0.025" length="0.25"/-->
+        <mesh filename = "package://bme_ros_simple_arm/meshes/forearm.dae"/>
       </geometry>
       <material name="orange"/>
@@ -145,7 +148,7 @@
     </visual>
   </link>
-  <gazebo reference="forearm_link">
+  <!--gazebo reference="forearm_link">
     <material>Gazebo/Orange</material>
-  </gazebo>
+  </gazebo-->
   <!-- Wrist joint -->
   <joint name="wrist_joint" type="revolute">
@@ -175,5 +178,6 @@
     <visual>
       <geometry>
-        <cylinder radius="0.02" length="0.1"/>
+        <!--cylinder radius="0.02" length="0.1"/-->
+        <mesh filename = "package://bme_ros_simple_arm/meshes/wrist.dae"/>
       </geometry>
       <material name="orange"/>
@@ -181,7 +185,7 @@
     </visual>
   </link>
-  <gazebo reference="wrist_link">
+  <!--gazebo reference="wrist_link">
     <material>Gazebo/Orange</material>
-  </gazebo>
+  </gazebo-->
   <!-- Gripper base joint -->
   <joint name="gripper_base_joint" type="fixed">

Commit message: increase wrist angle range

File: bme_ros_simple_arm/urdf/mogi_arm.xacro (robot description, xacro)
@@ -153,5 +153,5 @@
   <!-- Wrist joint -->
   <joint name="wrist_joint" type="revolute">
-    <limit lower="-1.5708" upper="1.5708" effort="54.0" velocity="3.14"/>
+    <limit lower="-2.3562" upper="2.3562" effort="54.0" velocity="3.14"/>
     <parent link="forearm_link"/>
     <child link="wrist_link"/>

Commit message: update urdf file to match with readme

File: bme_ros_simple_arm/urdf/mogi_arm.xacro (robot description, xacro)
@@ -1,10 +1,10 @@
 <?xml version="1.0"?>
 <robot name="mogi_arm" xmlns:xacro="http://www.ros.org/wiki/xacro">
+  <!-- RViz colors -->
+  <xacro:include filename="$(find bme_ros_simple_arm)/urdf/materials.xacro" />
   <!-- Transmisions -->
   <xacro:include filename="$(find bme_ros_simple_arm)/urdf/transmission.xacro" />
   <!-- Gazebo plugin -->
   <xacro:include filename="$(find bme_ros_simple_arm)/urdf/mogi_arm.gazebo" />
-  <!-- RViz colors -->
-  <xacro:include filename="$(find bme_ros_simple_arm)/urdf/materials.xacro" />
   <!-- Global reference link -->
   <link name="world"/>
@@ -67,6 +67,6 @@
     <visual>
       <geometry>
+        <mesh filename = "package://bme_ros_simple_arm/meshes/shoulder.dae"/>
         <!--cylinder radius="0.1" length="0.05"/-->
-        <mesh filename = "package://bme_ros_simple_arm/meshes/shoulder.dae"/>
       </geometry>
       <material name="orange"/>
@@ -104,6 +104,6 @@
     <visual>
       <geometry>
+        <mesh filename = "package://bme_ros_simple_arm/meshes/upper_arm.dae"/>
         <!--cylinder radius="0.05" length="0.2"/-->
-        <mesh filename = "package://bme_ros_simple_arm/meshes/upper_arm.dae"/>
       </geometry>
       <material name="orange"/>
@@ -141,6 +141,6 @@
     <visual>
       <geometry>
+        <mesh filename = "package://bme_ros_simple_arm/meshes/forearm.dae"/>
         <!--cylinder radius="0.025" length="0.25"/-->
-        <mesh filename = "package://bme_ros_simple_arm/meshes/forearm.dae"/>
       </geometry>
       <material name="orange"/>
@@ -178,6 +178,6 @@
     <visual>
       <geometry>
+        <mesh filename = "package://bme_ros_simple_arm/meshes/wrist.dae"/>
         <!--cylinder radius="0.02" length="0.1"/-->
-        <mesh filename = "package://bme_ros_simple_arm/meshes/wrist.dae"/>
       </geometry>
       <material name="orange"/>

Commit message: fake 6 axis to use KDL with the 4 axis robot

File: bme_ros_simple_arm/urdf/mogi_arm.xacro (robot description, xacro)
@@ -305,12 +305,15 @@
     <material>Gazebo/Blue</material>
   </gazebo>
-  <!-- End effector joint -->
-  <joint name="end_effector_joint" type="fixed">
+  <!-- Virtual roll joint -->
+  <joint name="virtual_roll_joint" type="revolute">
+    <limit lower="-1.57" upper="1.57" effort="54.0" velocity="3.14"/>
+    <parent link="wrist_link"/>
+    <child link="virtual_roll_link"/>
+    <axis xyz="0 0 1"/>
     <origin xyz="0.0 0.0 0.175" rpy="0 0 0"/>
-    <parent link="wrist_link"/>
-    <child link="end_effector_link"/>
-  </joint>
-  <!-- End effector link -->
-  <link name="end_effector_link">
+    <dynamics damping="0.0" friction="0.0"/>
+  </joint>
+  <!-- Virtual roll link -->
+  <link name="virtual_roll_link">
     <visual>
       <origin xyz="0 0 0" rpy="0 0 0"/>
@@ -328,4 +331,59 @@
     </inertial>
   </link>
+  <gazebo reference="virtual_roll_link">
+    <material>Gazebo/Red</material>
+  </gazebo>
+  <!-- Virtual yaw joint -->
+  <joint name="virtual_yaw_joint" type="revolute">
+    <limit lower="-1.57" upper="1.57" effort="54.0" velocity="3.14"/>
+    <parent link="virtual_roll_link"/>
+    <child link="virtual_yaw_link"/>
+    <axis xyz="1 0 0"/>
+    <origin xyz="0.0 0.0 0.0" rpy="0 0 0"/>
+    <dynamics damping="0.0" friction="0.0"/>
+  </joint>
+  <!-- Virtual yaw link -->
+  <link name="virtual_yaw_link">
+    <visual>
+      <origin xyz="0 0 0" rpy="0 0 0"/>
+      <geometry>
+        <box size="0.01 0.01 0.01" />
+      </geometry>
+      <material name="red"/>
+     </visual>
+    <inertial>
+      <origin xyz="0 0 0" />
+      <mass value="1.0e-03" />
+      <inertia ixx="1.0e-03" ixy="0.0" ixz="0.0"
+               iyy="1.0e-03" iyz="0.0"
+               izz="1.0e-03" />
+    </inertial>
+  </link>
+  <gazebo reference="virtual_yaw_link">
+    <material>Gazebo/Red</material>
+  </gazebo>
+  <!-- End effector joint -->
+  <joint name="end_effector_joint" type="fixed">
+    <origin xyz="0.0 0.0 0.0" rpy="0 0 0"/>
+    <parent link="virtual_yaw_link"/>
+    <child link="end_effector_link"/>
+  </joint>
+  <!-- End effector link -->
+  <link name="end_effector_link">
+    <visual>
+      <origin xyz="0 0 0" rpy="0 0 0"/>
+      <geometry>
+        <box size="0.01 0.01 0.01" />
+      </geometry>
+      <material name="red"/>
+     </visual>
+    <inertial>
+      <origin xyz="0 0 0" />
+      <mass value="1.0e-03" />
+      <inertia ixx="1.0e-03" ixy="0.0" ixz="0.0"
+               iyy="1.0e-03" iyz="0.0"
+               izz="1.0e-03" />
+    </inertial>
+  </link>
   <gazebo reference="end_effector_link">
     <material>Gazebo/Red</material>

File: bme_ros_simple_arm/urdf/transmission.xacro (robot description, xacro)
@@ -45,4 +45,26 @@
     </actuator>
   </transmission>
+  <!-- Virtual roll transmission -->
+  <transmission name ="virtual_roll_trans">
+    <type>transmission_interface/SimpleTransmission</type>
+    <joint name="virtual_roll_joint">
+      <hardwareInterface>hardware_interface/PositionJointInterface</hardwareInterface>
+    </joint>
+    <actuator name="virtual_roll_motor">
+      <hardwareInterface>hardware_interface/PositionJointInterface</hardwareInterface>
+      <mechanicalReduction>1</mechanicalReduction>
+    </actuator>
+  </transmission>
+  <!-- Virtual yaw transmission -->
+  <transmission name ="virtual_yaw">
+    <type>transmission_interface/SimpleTransmission</type>
+    <joint name="virtual_yaw_joint">
+      <hardwareInterface>hardware_interface/PositionJointInterface</hardwareInterface>
+    </joint>
+    <actuator name="virtual_yaw_motor">
+      <hardwareInterface>hardware_interface/PositionJointInterface</hardwareInterface>
+      <mechanicalReduction>1</mechanicalReduction>
+    </actuator>
+  </transmission>
   <!-- Left finger transmission -->
   <transmission name ="left_finger_trans">

Commit message: increase angle range of virtual joints

File: bme_ros_simple_arm/urdf/mogi_arm.xacro (robot description, xacro)
@@ -307,5 +307,5 @@
   <!-- Virtual roll joint -->
   <joint name="virtual_roll_joint" type="revolute">
-    <limit lower="-1.57" upper="1.57" effort="54.0" velocity="3.14"/>
+    <limit lower="-3.1415" upper="3.1415" effort="54.0" velocity="3.14"/>
     <parent link="wrist_link"/>
     <child link="virtual_roll_link"/>
@@ -336,5 +336,5 @@
   <!-- Virtual yaw joint -->
   <joint name="virtual_yaw_joint" type="revolute">
-    <limit lower="-1.57" upper="1.57" effort="54.0" velocity="3.14"/>
+    <limit lower="-3.1415" upper="3.1415" effort="54.0" velocity="3.14"/>
     <parent link="virtual_roll_link"/>
     <child link="virtual_yaw_link"/>
