Commit message: update to 6 DoF moveit config

File: bme_ros2_simple_arm_moveit_config/config/mogi_arm.ros2_control.xacro (robot description, xacro)
@@ -36,4 +36,18 @@
                 <state_interface name="velocity"/>
             </joint>
+            <joint name="virtual_roll_joint">
+                <command_interface name="position"/>
+                <state_interface name="position">
+                  <param name="initial_value">${initial_positions['virtual_roll_joint']}</param>
+                </state_interface>
+                <state_interface name="velocity"/>
+            </joint>
+            <joint name="virtual_yaw_joint">
+                <command_interface name="position"/>
+                <state_interface name="position">
+                  <param name="initial_value">${initial_positions['virtual_yaw_joint']}</param>
+                </state_interface>
+                <state_interface name="velocity"/>
+            </joint>
             <joint name="left_finger_joint">
                 <command_interface name="position"/>
