Commit message: add shoulder joints to urdf, add joint state publisher and forward message with gz bridge

File: bme_ros2_simple_arm/urdf/mogi_arm.xacro (robot description, xacro)
@@ -2,5 +2,7 @@
 <robot name="mogi_arm" xmlns:xacro="http://www.ros.org/wiki/xacro">
   <!-- STEP 3 - RViz colors -->
-  <xacro:include filename="$(find bme_ros2_navigation)/urdf/materials.xacro" />
+  <xacro:include filename="$(find bme_ros2_simple_arm)/urdf/materials.xacro" />
+  <!-- STEP 5 - Gazebo plugin -->
+  <xacro:include filename="$(find bme_ros2_simple_arm)/urdf/mogi_arm.gazebo" />
   <!-- STEP 1 - Global reference link -->
   <link name="world"/>
@@ -33,3 +35,69 @@
     </visual>
   </link>
+  <!-- STEP 4 - Shoulder pan joint -->
+  <joint name="shoulder_pan_joint" type="revolute">
+    <limit lower="-3.14" upper="3.14" effort="330.0" velocity="3.14"/>
+    <parent link="base_link"/>
+    <child link="shoulder_link"/>
+    <axis xyz="0 0 1"/>
+    <origin xyz="0.0 0.0 0.05" rpy="0.0 0.0 0.0"/>
+    <dynamics damping="0.0" friction="0.0"/>
+  </joint>
+  <!-- Shoulder link -->
+  <link name="shoulder_link">
+    <inertial>
+      <mass value="0.5"/>
+      <origin xyz="0.0 0.0 0.0" rpy="0.0 0.0 0.0"/>
+      <inertia ixx="0.0014" ixy="0.0" ixz="0.0"
+               iyy="0.0014" iyz="0.0"
+               izz="0.0025"
+      />
+    </inertial>
+    <collision>
+      <geometry>
+        <cylinder radius="0.1" length="0.05"/>
+      </geometry>
+      <origin xyz="0.0 0.0 0.0" rpy="0.0 0.0 0.0"/>
+    </collision>
+    <visual>
+      <geometry>
+        <cylinder radius="0.1" length="0.05"/>
+      </geometry>
+      <material name="orange"/>
+      <origin xyz="0.0 0.0 0.0" rpy="0.0 0.0 0.0"/>
+    </visual>
+  </link>
+  <!-- Shoulder lift joint -->
+  <joint name="shoulder_lift_joint" type="revolute">
+    <limit lower="-1.5708" upper="1.5708" effort="330.0" velocity="3.14"/>
+    <parent link="shoulder_link"/>
+    <child link="upper_arm_link"/>
+    <axis xyz="0 1 0"/>
+    <origin xyz="0.0 0.0 0.025" rpy="0.0 0.0 0.0"/>
+    <dynamics damping="0.0" friction="0.0"/>
+  </joint>
+  <!-- Upper arm link -->
+  <link name="upper_arm_link">
+    <inertial>
+      <mass value="0.3"/>
+      <origin xyz="0.0 0.0 0.1" rpy="0.0 0.0 0.0"/>
+      <inertia ixx="0.0012" ixy="0.0" ixz="0.0"
+               iyy="0.0012" iyz="0.0"
+               izz="0.0004"
+      />
+    </inertial>
+    <collision>
+      <geometry>
+        <cylinder radius="0.05" length="0.2"/>
+      </geometry>
+      <origin xyz="0.0 0.0 0.1" rpy="0.0 0.0 0.0"/>
+    </collision>
+    <visual>
+      <geometry>
+        <cylinder radius="0.05" length="0.2"/>
+      </geometry>
+      <material name="orange"/>
+      <origin xyz="0.0 0.0 0.1" rpy="0.0 0.0 0.0"/>
+    </visual>
+  </link>
 </robot>

Commit message: add remaining joints and gripper

File: bme_ros2_simple_arm/urdf/mogi_arm.xacro (robot description, xacro)
@@ -101,3 +101,181 @@
     </visual>
   </link>
+  <!-- STEP 6 - Elbow joint -->
+  <joint name="elbow_joint" type="revolute">
+    <limit lower="-2.3562" upper="2.3562" effort="150.0" velocity="3.14"/>
+    <parent link="upper_arm_link"/>
+    <child link="forearm_link"/>
+    <axis xyz="0 1 0"/>
+    <origin xyz="0.0 0.0 0.2" rpy="0.0 0.0 0.0"/>
+    <dynamics damping="0.0" friction="0.0"/>
+  </joint>
+  <!-- Forearm link -->
+  <link name="forearm_link">
+    <inertial>
+      <mass value="0.2"/>
+      <origin xyz="0.0 0.0 0.125" rpy="0.0 0.0 0.0"/>
+      <inertia ixx="0.0011" ixy="0.0" ixz="0.0"
+               iyy="0.0011" iyz="0.0"
+               izz="0.0004"
+      />
+    </inertial>
+    <collision>
+      <geometry>
+        <cylinder radius="0.025" length="0.25"/>
+      </geometry>
+      <origin xyz="0.0 0.0 0.125" rpy="0.0 0.0 0.0"/>
+    </collision>
+    <visual>
+      <geometry>
+        <cylinder radius="0.025" length="0.25"/>
+      </geometry>
+      <material name="orange"/>
+      <origin xyz="0.0 0.0 0.125" rpy="0.0 0.0 0.0"/>
+    </visual>
+  </link>
+  <!-- STEP 7 - Wrist joint -->
+  <joint name="wrist_joint" type="revolute">
+    <limit lower="-2.3562" upper="2.3562" effort="54.0" velocity="3.14"/>
+    <parent link="forearm_link"/>
+    <child link="wrist_link"/>
+    <axis xyz="0 1 0"/>
+    <origin xyz="0.0 0.0 0.25" rpy="0.0 0.0 0.0"/>
+    <dynamics damping="0.0" friction="0.0"/>
+  </joint>
+  <!-- Wrist link -->
+  <link name="wrist_link">
+    <inertial>
+      <mass value="0.1"/>
+      <origin xyz="0.0 0.0 0.05" rpy="0.0 0.0 0.0"/>
+      <inertia ixx="0.00009" ixy="0.0" ixz="0.0"
+               iyy="0.00009" iyz="0.0"
+               izz="0.00002"
+      />
+    </inertial>
+    <collision>
+      <geometry>
+        <cylinder radius="0.02" length="0.1"/>
+      </geometry>
+      <origin xyz="0.0 0.0 0.05" rpy="0.0 0.0 0.0"/>
+    </collision>
+    <visual>
+      <geometry>
+        <cylinder radius="0.02" length="0.1"/>
+      </geometry>
+      <material name="orange"/>
+      <origin xyz="0.0 0.0 0.05" rpy="0.0 0.0 0.0"/>
+    </visual>
+  </link>
+  <!-- STEP 8 - Gripper base joint -->
+  <joint name="gripper_base_joint" type="fixed">
+    <parent link="wrist_link"/>
+    <child link="gripper_base"/>
+    <origin xyz="0.0 0 0.105" rpy="0.0 0 0"/>
+  </joint>
+  <!-- Gripper base link -->
+  <link name="gripper_base">
+    <inertial>
+      <mass value="0.1"/>
+      <origin xyz="0.0 0.0 0.0" rpy="0.0 0.0 0.0"/>
+      <inertia ixx="0.00009" ixy="0.0" ixz="0.0"
+               iyy="0.00009" iyz="0.0"
+               izz="0.00002"
+      />
+    </inertial>
+    <collision>
+      <geometry>
+        <box size=".05 .1 .01"/>
+      </geometry>
+      <origin xyz="0.0 0.0 0.0" rpy="0.0 0.0 0.0"/>
+    </collision>
+    <visual>
+      <geometry>
+        <box size=".05 .1 .01"/>
+      </geometry>
+      <material name="grey"/>
+      <origin xyz="0.0 0.0 0.0" rpy="0.0 0.0 0.0"/>
+    </visual>
+  </link>
+  <!-- Left finger joint -->
+  <joint name="left_finger_joint" type="prismatic">
+    <limit lower="0" upper="0.04" effort="100.0" velocity="4.0"/>
+    <parent link="gripper_base"/>
+    <child link="left_finger"/>
+    <axis xyz="0 1 0"/>
+    <origin xyz="0.0 0.01 0.045" />
+  </joint>
+  <!-- Left finger link -->
+  <link name="left_finger">
+    <inertial>
+      <mass value="0.1"/>
+      <origin xyz="0.0 0.0 0.0" rpy="0.0 0.0 0.0"/>
+      <inertia ixx="0.00009" ixy="0.0" ixz="0.0"
+               iyy="0.00009" iyz="0.0"
+               izz="0.00002"
+      />
+    </inertial>
+    <collision>
+      <geometry>
+        <box size=".04 .01 .08"/>
+      </geometry>
+      <origin xyz="0.0 0.0 0.0" rpy="0.0 0.0 0.0"/>
+    </collision>
+    <visual>
+      <geometry>
+        <box size=".04 .01 .08"/>
+      </geometry>
+      <material name="blue"/>
+      <origin xyz="0.0 0.0 0.0" rpy="0.0 0.0 0.0"/>
+    </visual>
+  </link>
+  <gazebo reference="left_finger">
+    <kp>1000000.0</kp>
+    <kd>100.0</kd>
+    <mu1>15</mu1>
+    <mu2>15</mu2>
+    <fdir1>1 0 0</fdir1>
+    <maxVel>1.0</maxVel>
+    <minDepth>0.002</minDepth>
+  </gazebo>
+  <!-- Right finger joint -->
+  <joint name="right_finger_joint" type="prismatic">
+    <limit lower="0" upper="0.04" effort="100.0" velocity="4.0"/>
+    <parent link="gripper_base"/>
+    <child link="right_finger"/>
+    <axis xyz="0 -1 0"/>
+    <origin xyz="0.0 -0.01 0.045" />
+  </joint>
+  <!-- Right finger link -->
+  <link name="right_finger">
+    <inertial>
+      <mass value="0.1"/>
+      <origin xyz="0.0 0.0 0.0" rpy="0.0 0.0 0.0"/>
+      <inertia ixx="0.00009" ixy="0.0" ixz="0.0"
+               iyy="0.00009" iyz="0.0"
+               izz="0.00002"
+      />
+    </inertial>
+    <collision>
+      <geometry>
+        <box size=".04 .01 .08"/>
+      </geometry>
+      <origin xyz="0.0 0.0 0.0" rpy="0.0 0.0 0.0"/>
+    </collision>
+    <visual>
+      <geometry>
+        <box size=".04 .01 .08"/>
+      </geometry>
+      <material name="blue"/>
+      <origin xyz="0.0 0.0 0.0" rpy="0.0 0.0 0.0"/>
+    </visual>
+  </link>
+  <gazebo reference="right_finger">
+    <kp>1000000.0</kp>
+    <kd>100.0</kd>
+    <mu1>15</mu1>
+    <mu2>15</mu2>
+    <fdir1>1 0 0</fdir1>
+    <maxVel>1.0</maxVel>
+    <minDepth>0.002</minDepth>
+  </gazebo>
 </robot>

Commit message: Add gz_ros2_control to control joint trajectory

File: bme_ros2_simple_arm/urdf/mogi_arm.xacro (robot description, xacro)
@@ -279,3 +279,74 @@
     <minDepth>0.002</minDepth>
   </gazebo>
+  <ros2_control name="GazeboSystem" type="system">
+    <hardware>
+      <plugin>gz_ros2_control/GazeboSimSystem</plugin>
+    </hardware>
+    <joint name="shoulder_pan_joint">
+      <command_interface name="position">
+        <param name="min">-2</param>
+        <param name="max">2</param>
+      </command_interface>
+      <state_interface name="position">
+        <param name="initial_value">0.0</param>
+      </state_interface>
+      <state_interface name="velocity"/>
+      <state_interface name="effort"/>
+    </joint>
+    <joint name="shoulder_lift_joint">
+      <command_interface name="position">
+        <param name="min">-2</param>
+        <param name="max">2</param>
+      </command_interface>
+      <state_interface name="position">
+        <param name="initial_value">0.0</param>
+      </state_interface>
+      <state_interface name="velocity"/>
+      <state_interface name="effort"/>
+    </joint>
+    <joint name="elbow_joint">
+      <command_interface name="position">
+        <param name="min">-2</param>
+        <param name="max">2</param>
+      </command_interface>
+      <state_interface name="position">
+        <param name="initial_value">0.0</param>
+      </state_interface>
+      <state_interface name="velocity"/>
+      <state_interface name="effort"/>
+    </joint>
+    <joint name="wrist_joint">
+      <command_interface name="position">
+        <param name="min">-2</param>
+        <param name="max">2</param>
+      </command_interface>
+      <state_interface name="position">
+        <param name="initial_value">0.0</param>
+      </state_interface>
+      <state_interface name="velocity"/>
+      <state_interface name="effort"/>
+    </joint>
+    <joint name="left_finger_joint">
+      <command_interface name="position">
+        <param name="min">-2</param>
+        <param name="max">2</param>
+      </command_interface>
+      <state_interface name="position">
+        <param name="initial_value">0.0</param>
+      </state_interface>
+      <state_interface name="velocity"/>
+      <state_interface name="effort"/>
+    </joint>
+    <joint name="right_finger_joint">
+      <command_interface name="position">
+        <param name="min">-2</param>
+        <param name="max">2</param>
+      </command_interface>
+      <state_interface name="position">
+        <param name="initial_value">0.0</param>
+      </state_interface>
+      <state_interface name="velocity"/>
+      <state_interface name="effort"/>
+    </joint>
+  </ros2_control>
 </robot>

Commit message: replace link models with 3D models

File: bme_ros2_simple_arm/urdf/mogi_arm.xacro (robot description, xacro)
@@ -62,5 +62,6 @@
     <visual>
       <geometry>
-        <cylinder radius="0.1" length="0.05"/>
+        <!-- <cylinder radius="0.1" length="0.05"/> -->
+        <mesh filename = "package://bme_ros2_simple_arm/meshes/shoulder.dae"/>
       </geometry>
       <material name="orange"/>
@@ -95,5 +96,6 @@
     <visual>
       <geometry>
-        <cylinder radius="0.05" length="0.2"/>
+        <!-- <cylinder radius="0.05" length="0.2"/> -->
+        <mesh filename = "package://bme_ros2_simple_arm/meshes/upper_arm.dae"/>
       </geometry>
       <material name="orange"/>
@@ -128,5 +130,6 @@
     <visual>
       <geometry>
-        <cylinder radius="0.025" length="0.25"/>
+        <!-- <cylinder radius="0.025" length="0.25"/> -->
+        <mesh filename = "package://bme_ros2_simple_arm/meshes/forearm.dae"/>
       </geometry>
       <material name="orange"/>
@@ -161,5 +164,6 @@
     <visual>
       <geometry>
-        <cylinder radius="0.02" length="0.1"/>
+        <!-- <cylinder radius="0.02" length="0.1"/> -->
+        <mesh filename = "package://bme_ros2_simple_arm/meshes/wrist.dae"/>
       </geometry>
       <material name="orange"/>

Commit message: add end effector link and cleanup urdf

File: bme_ros2_simple_arm/urdf/mogi_arm.xacro (robot description, xacro)
@@ -35,5 +35,5 @@
     </visual>
   </link>
-  <!-- STEP 4 - Shoulder pan joint -->
+  <!-- STEP 4 - Shoulder -->
   <joint name="shoulder_pan_joint" type="revolute">
     <limit lower="-3.14" upper="3.14" effort="330.0" velocity="3.14"/>
@@ -103,5 +103,5 @@
     </visual>
   </link>
-  <!-- STEP 6 - Elbow joint -->
+  <!-- STEP 6 - Elbow -->
   <joint name="elbow_joint" type="revolute">
     <limit lower="-2.3562" upper="2.3562" effort="150.0" velocity="3.14"/>
@@ -137,5 +137,5 @@
     </visual>
   </link>
-  <!-- STEP 7 - Wrist joint -->
+  <!-- STEP 7 - Wrist -->
   <joint name="wrist_joint" type="revolute">
     <limit lower="-2.3562" upper="2.3562" effort="54.0" velocity="3.14"/>
@@ -171,5 +171,5 @@
     </visual>
   </link>
-  <!-- STEP 8 - Gripper base joint -->
+  <!-- STEP 8 - Gripper -->
   <joint name="gripper_base_joint" type="fixed">
     <parent link="wrist_link"/>
@@ -283,4 +283,5 @@
     <minDepth>0.002</minDepth>
   </gazebo>
+  <!-- STEP 9 - ROS2 control -->
   <ros2_control name="GazeboSystem" type="system">
     <hardware>
@@ -354,3 +355,26 @@
     </joint>
   </ros2_control>
+  <!-- STEP 10 - End effector -->
+  <joint name="end_effector_joint" type="fixed">
+    <origin xyz="0.0 0.0 0.175" rpy="0 0 0"/>
+    <parent link="wrist_link"/>
+    <child link="end_effector_link"/>
+  </joint>
+  <!-- End effector link -->
+  <link name="end_effector_link">
+    <visual>
+      <origin xyz="0 0 0" rpy="0 0 0"/>
+      <geometry>
+        <box size="0.01 0.01 0.01" />
+      </geometry>
+      <material name="red"/>
+     </visual>
+    <inertial>
+      <origin xyz="0 0 0" />
+      <mass value="1.0e-03" />
+      <inertia ixx="1.0e-03" ixy="0.0" ixz="0.0"
+               iyy="1.0e-03" iyz="0.0"
+               izz="1.0e-03" />
+    </inertial>
+  </link>
 </robot>

Commit message: readme completed till ROS control

File: bme_ros2_simple_arm/urdf/mogi_arm.xacro (robot description, xacro)
@@ -3,5 +3,5 @@
   <!-- STEP 3 - RViz colors -->
   <xacro:include filename="$(find bme_ros2_simple_arm)/urdf/materials.xacro" />
-  <!-- STEP 5 - Gazebo plugin -->
+  <!-- STEP 8 - Gazebo plugin -->
   <xacro:include filename="$(find bme_ros2_simple_arm)/urdf/mogi_arm.gazebo" />
   <!-- STEP 1 - Global reference link -->
@@ -62,6 +62,5 @@
     <visual>
       <geometry>
-        <!-- <cylinder radius="0.1" length="0.05"/> -->
-        <mesh filename = "package://bme_ros2_simple_arm/meshes/shoulder.dae"/>
+        <cylinder radius="0.1" length="0.05"/>
       </geometry>
       <material name="orange"/>
@@ -96,6 +95,5 @@
     <visual>
       <geometry>
-        <!-- <cylinder radius="0.05" length="0.2"/> -->
-        <mesh filename = "package://bme_ros2_simple_arm/meshes/upper_arm.dae"/>
+        <cylinder radius="0.05" length="0.2"/>
       </geometry>
       <material name="orange"/>
@@ -103,5 +101,5 @@
     </visual>
   </link>
-  <!-- STEP 6 - Elbow -->
+  <!-- STEP 5 - Elbow -->
   <joint name="elbow_joint" type="revolute">
     <limit lower="-2.3562" upper="2.3562" effort="150.0" velocity="3.14"/>
@@ -130,6 +128,5 @@
     <visual>
       <geometry>
-        <!-- <cylinder radius="0.025" length="0.25"/> -->
-        <mesh filename = "package://bme_ros2_simple_arm/meshes/forearm.dae"/>
+        <cylinder radius="0.025" length="0.25"/>
       </geometry>
       <material name="orange"/>
@@ -137,5 +134,5 @@
     </visual>
   </link>
-  <!-- STEP 7 - Wrist -->
+  <!-- STEP 6 - Wrist -->
   <joint name="wrist_joint" type="revolute">
     <limit lower="-2.3562" upper="2.3562" effort="54.0" velocity="3.14"/>
@@ -164,6 +161,5 @@
     <visual>
       <geometry>
-        <!-- <cylinder radius="0.02" length="0.1"/> -->
-        <mesh filename = "package://bme_ros2_simple_arm/meshes/wrist.dae"/>
+        <cylinder radius="0.02" length="0.1"/>
       </geometry>
       <material name="orange"/>
@@ -171,5 +167,5 @@
     </visual>
   </link>
-  <!-- STEP 8 - Gripper -->
+  <!-- STEP 7 - Gripper -->
   <joint name="gripper_base_joint" type="fixed">
     <parent link="wrist_link"/>
@@ -283,98 +279,3 @@
     <minDepth>0.002</minDepth>
   </gazebo>
-  <!-- STEP 9 - ROS2 control -->
-  <ros2_control name="GazeboSystem" type="system">
-    <hardware>
-      <plugin>gz_ros2_control/GazeboSimSystem</plugin>
-    </hardware>
-    <joint name="shoulder_pan_joint">
-      <command_interface name="position">
-        <param name="min">-2</param>
-        <param name="max">2</param>
-      </command_interface>
-      <state_interface name="position">
-        <param name="initial_value">0.0</param>
-      </state_interface>
-      <state_interface name="velocity"/>
-      <state_interface name="effort"/>
-    </joint>
-    <joint name="shoulder_lift_joint">
-      <command_interface name="position">
-        <param name="min">-2</param>
-        <param name="max">2</param>
-      </command_interface>
-      <state_interface name="position">
-        <param name="initial_value">0.0</param>
-      </state_interface>
-      <state_interface name="velocity"/>
-      <state_interface name="effort"/>
-    </joint>
-    <joint name="elbow_joint">
-      <command_interface name="position">
-        <param name="min">-2</param>
-        <param name="max">2</param>
-      </command_interface>
-      <state_interface name="position">
-        <param name="initial_value">0.0</param>
-      </state_interface>
-      <state_interface name="velocity"/>
-      <state_interface name="effort"/>
-    </joint>
-    <joint name="wrist_joint">
-      <command_interface name="position">
-        <param name="min">-2</param>
-        <param name="max">2</param>
-      </command_interface>
-      <state_interface name="position">
-        <param name="initial_value">0.0</param>
-      </state_interface>
-      <state_interface name="velocity"/>
-      <state_interface name="effort"/>
-    </joint>
-    <joint name="left_finger_joint">
-      <command_interface name="position">
-        <param name="min">-2</param>
-        <param name="max">2</param>
-      </command_interface>
-      <state_interface name="position">
-        <param name="initial_value">0.0</param>
-      </state_interface>
-      <state_interface name="velocity"/>
-      <state_interface name="effort"/>
-    </joint>
-    <joint name="right_finger_joint">
-      <command_interface name="position">
-        <param name="min">-2</param>
-        <param name="max">2</param>
-      </command_interface>
-      <state_interface name="position">
-        <param name="initial_value">0.0</param>
-      </state_interface>
-      <state_interface name="velocity"/>
-      <state_interface name="effort"/>
-    </joint>
-  </ros2_control>
-  <!-- STEP 10 - End effector -->
-  <joint name="end_effector_joint" type="fixed">
-    <origin xyz="0.0 0.0 0.175" rpy="0 0 0"/>
-    <parent link="wrist_link"/>
-    <child link="end_effector_link"/>
-  </joint>
-  <!-- End effector link -->
-  <link name="end_effector_link">
-    <visual>
-      <origin xyz="0 0 0" rpy="0 0 0"/>
-      <geometry>
-        <box size="0.01 0.01 0.01" />
-      </geometry>
-      <material name="red"/>
-     </visual>
-    <inertial>
-      <origin xyz="0 0 0" />
-      <mass value="1.0e-03" />
-      <inertia ixx="1.0e-03" ixy="0.0" ixz="0.0"
-               iyy="1.0e-03" iyz="0.0"
-               izz="1.0e-03" />
-    </inertial>
-  </link>
 </robot>

Commit message: add joint trajectory controller

File: bme_ros2_simple_arm/urdf/mogi_arm.xacro (robot description, xacro)
@@ -279,3 +279,75 @@
     <minDepth>0.002</minDepth>
   </gazebo>
+  <!-- STEP 9 - ROS2 control -->
+  <ros2_control name="GazeboSystem" type="system">
+    <hardware>
+      <plugin>gz_ros2_control/GazeboSimSystem</plugin>
+    </hardware>
+    <joint name="shoulder_pan_joint">
+      <command_interface name="position">
+        <param name="min">-2</param>
+        <param name="max">2</param>
+      </command_interface>
+      <state_interface name="position">
+        <param name="initial_value">0.0</param>
+      </state_interface>
+      <state_interface name="velocity"/>
+      <state_interface name="effort"/>
+    </joint>
+    <joint name="shoulder_lift_joint">
+      <command_interface name="position">
+        <param name="min">-2</param>
+        <param name="max">2</param>
+      </command_interface>
+      <state_interface name="position">
+        <param name="initial_value">0.0</param>
+      </state_interface>
+      <state_interface name="velocity"/>
+      <state_interface name="effort"/>
+    </joint>
+    <joint name="elbow_joint">
+      <command_interface name="position">
+        <param name="min">-2</param>
+        <param name="max">2</param>
+      </command_interface>
+      <state_interface name="position">
+        <param name="initial_value">0.0</param>
+      </state_interface>
+      <state_interface name="velocity"/>
+      <state_interface name="effort"/>
+    </joint>
+    <joint name="wrist_joint">
+      <command_interface name="position">
+        <param name="min">-2</param>
+        <param name="max">2</param>
+      </command_interface>
+      <state_interface name="position">
+        <param name="initial_value">0.0</param>
+      </state_interface>
+      <state_interface name="velocity"/>
+      <state_interface name="effort"/>
+    </joint>
+    <joint name="left_finger_joint">
+      <command_interface name="position">
+        <param name="min">-2</param>
+        <param name="max">2</param>
+      </command_interface>
+      <state_interface name="position">
+        <param name="initial_value">0.0</param>
+      </state_interface>
+      <state_interface name="velocity"/>
+      <state_interface name="effort"/>
+    </joint>
+    <joint name="right_finger_joint">
+      <command_interface name="position">
+        <param name="min">-2</param>
+        <param name="max">2</param>
+      </command_interface>
+      <state_interface name="position">
+        <param name="initial_value">0.0</param>
+      </state_interface>
+      <state_interface name="velocity"/>
+      <state_interface name="effort"/>
+    </joint>
+  </ros2_control>
 </robot>
