Commit message: add contact sensor, detachable links and end effector

File: bme_ros2_simple_arm/urdf/mogi_arm.xacro (robot description, xacro)
@@ -62,5 +62,6 @@
     <visual>
       <geometry>
-        <cylinder radius="0.1" length="0.05"/>
+        <!-- <cylinder radius="0.1" length="0.05"/> -->
+        <mesh filename = "package://bme_ros2_simple_arm/meshes/shoulder.dae"/>
       </geometry>
       <material name="orange"/>
@@ -95,5 +96,6 @@
     <visual>
       <geometry>
-        <cylinder radius="0.05" length="0.2"/>
+        <!-- <cylinder radius="0.05" length="0.2"/> -->
+        <mesh filename = "package://bme_ros2_simple_arm/meshes/upper_arm.dae"/>
       </geometry>
       <material name="orange"/>
@@ -128,5 +130,6 @@
     <visual>
       <geometry>
-        <cylinder radius="0.025" length="0.25"/>
+        <!-- <cylinder radius="0.025" length="0.25"/> -->
+        <mesh filename = "package://bme_ros2_simple_arm/meshes/forearm.dae"/>
       </geometry>
       <material name="orange"/>
@@ -161,5 +164,6 @@
     <visual>
       <geometry>
-        <cylinder radius="0.02" length="0.1"/>
+        <!-- <cylinder radius="0.02" length="0.1"/> -->
+        <mesh filename = "package://bme_ros2_simple_arm/meshes/wrist.dae"/>
       </geometry>
       <material name="orange"/>
@@ -351,3 +355,26 @@
     </joint>
   </ros2_control>
+  <!-- STEP 10 - End effector -->
+  <joint name="end_effector_joint" type="fixed">
+    <origin xyz="0.0 0.0 0.175" rpy="0 0 0"/>
+    <parent link="wrist_link"/>
+    <child link="end_effector_link"/>
+  </joint>
+  <!-- End effector link -->
+  <link name="end_effector_link">
+    <visual>
+      <origin xyz="0 0 0" rpy="0 0 0"/>
+      <geometry>
+        <box size="0.01 0.01 0.01" />
+      </geometry>
+      <material name="red"/>
+     </visual>
+    <inertial>
+      <origin xyz="0 0 0" />
+      <mass value="1.0e-03" />
+      <inertia ixx="1.0e-03" ixy="0.0" ixz="0.0"
+               iyy="1.0e-03" iyz="0.0"
+               izz="1.0e-03" />
+    </inertial>
+  </link>
 </robot>

Commit message: add gripper and table camera

File: bme_ros2_simple_arm/urdf/mogi_arm.xacro (robot description, xacro)
@@ -378,3 +378,67 @@
     </inertial>
   </link>
+  <!-- STEP 11 - Gripper camera -->
+  <joint type="fixed" name="gripper_camera_joint">
+    <origin xyz="0.0 0.0 0.0" rpy="0 -1.5707 0"/>
+    <child link="gripper_camera_link"/>
+    <parent link="gripper_base"/>
+  </joint>
+  <link name='gripper_camera_link'>
+    <pose>0 0 0 0 0 0</pose>
+    <inertial>
+      <mass value="1.0e-03"/>
+      <origin xyz="0 0 0" rpy="0 0 0"/>
+      <inertia
+          ixx="1e-6" ixy="0" ixz="0"
+          iyy="1e-6" iyz="0"
+          izz="1e-6"
+      />
+    </inertial>
+    <visual>
+      <origin xyz="0 0 0" rpy="0 0 0"/>
+      <geometry>
+        <box size=".01 .01 .01"/>
+      </geometry>
+      <material name="red"/>
+    </visual>
+  </link>
+  <joint type="fixed" name="gripper_camera_optical_joint">
+    <origin xyz="0 0 0" rpy="-1.5707 0 -1.5707"/>
+    <child link="gripper_camera_link_optical"/>
+    <parent link="gripper_camera_link"/>
+  </joint>
+  <link name="gripper_camera_link_optical">
+  </link>
+  <!-- STEP 12 - Table camera -->
+  <joint type="fixed" name="table_camera_joint">
+    <origin xyz="1.0 0.4 0.2" rpy="0 0 3.6652"/>
+    <child link="table_camera_link"/>
+    <parent link="world"/>
+  </joint>
+  <link name='table_camera_link'>
+    <pose>0 0 0 0 0 0</pose>
+    <inertial>
+      <mass value="1.0e-03"/>
+      <origin xyz="0 0 0" rpy="0 0 0"/>
+      <inertia
+          ixx="1e-6" ixy="0" ixz="0"
+          iyy="1e-6" iyz="0"
+          izz="1e-6"
+      />
+    </inertial>
+    <visual>
+      <origin xyz="0 0 0" rpy="0 0 0"/>
+      <geometry>
+        <box size=".05 .05 .05"/>
+      </geometry>
+      <material name="red"/>
+    </visual>
+  </link>
+  <joint type="fixed" name="table_camera_optical_joint">
+    <origin xyz="0 0 0" rpy="-1.5707 0 -1.5707"/>
+    <child link="table_camera_link_optical"/>
+    <parent link="table_camera_link"/>
+  </joint>
+  <link name="table_camera_link_optical">
+  </link>
 </robot>

Commit message: Add fake 6 DoF changes to the robot

File: bme_ros2_simple_arm/urdf/mogi_arm.xacro (robot description, xacro)
@@ -283,4 +283,56 @@
     <minDepth>0.002</minDepth>
   </gazebo>
+  <!-- STEP 13 - Virtual roll joint -->
+  <joint name="virtual_roll_joint" type="revolute">
+    <limit lower="-3.1415" upper="3.1415" effort="54.0" velocity="3.14"/>
+    <parent link="wrist_link"/>
+    <child link="virtual_roll_link"/>
+    <axis xyz="0 0 1"/>
+    <origin xyz="0.0 0.0 0.175" rpy="0 0 0"/>
+    <dynamics damping="0.0" friction="0.0"/>
+  </joint>
+  <!-- Virtual roll link -->
+  <link name="virtual_roll_link">
+    <visual>
+      <origin xyz="0 0 0" rpy="0 0 0"/>
+      <geometry>
+        <box size="0.01 0.01 0.01" />
+      </geometry>
+      <material name="red"/>
+     </visual>
+    <inertial>
+      <origin xyz="0 0 0" />
+      <mass value="1.0e-03" />
+      <inertia ixx="1.0e-03" ixy="0.0" ixz="0.0"
+               iyy="1.0e-03" iyz="0.0"
+               izz="1.0e-03" />
+    </inertial>
+  </link>
+  <!-- Virtual yaw joint -->
+  <joint name="virtual_yaw_joint" type="revolute">
+    <limit lower="-3.1415" upper="3.1415" effort="54.0" velocity="3.14"/>
+    <parent link="virtual_roll_link"/>
+    <child link="virtual_yaw_link"/>
+    <axis xyz="1 0 0"/>
+    <origin xyz="0.0 0.0 0.0" rpy="0 0 0"/>
+    <dynamics damping="0.0" friction="0.0"/>
+  </joint>
+  <!-- Virtual yaw link -->
+  <link name="virtual_yaw_link">
+    <visual>
+      <origin xyz="0 0 0" rpy="0 0 0"/>
+      <geometry>
+        <box size="0.01 0.01 0.01" />
+      </geometry>
+      <material name="red"/>
+     </visual>
+    <inertial>
+      <origin xyz="0 0 0" />
+      <mass value="1.0e-03" />
+      <inertia ixx="1.0e-03" ixy="0.0" ixz="0.0"
+               iyy="1.0e-03" iyz="0.0"
+               izz="1.0e-03" />
+    </inertial>
+  </link>
   <!-- STEP 9 - ROS2 control -->
   <ros2_control name="GazeboSystem" type="system">
@@ -332,4 +384,26 @@
       <state_interface name="effort"/>
     </joint>
+    <joint name="virtual_roll_joint">
+      <command_interface name="position">
+        <param name="min">-2</param>
+        <param name="max">2</param>
+      </command_interface>
+      <state_interface name="position">
+        <param name="initial_value">0.0</param>
+      </state_interface>
+      <state_interface name="velocity"/>
+      <state_interface name="effort"/>
+    </joint>
+    <joint name="virtual_yaw_joint">
+      <command_interface name="position">
+        <param name="min">-2</param>
+        <param name="max">2</param>
+      </command_interface>
+      <state_interface name="position">
+        <param name="initial_value">0.0</param>
+      </state_interface>
+      <state_interface name="velocity"/>
+      <state_interface name="effort"/>
+    </joint>
     <joint name="left_finger_joint">
       <command_interface name="position">
@@ -358,5 +432,5 @@
   <joint name="end_effector_joint" type="fixed">
     <origin xyz="0.0 0.0 0.175" rpy="0 0 0"/>
-    <parent link="wrist_link"/>
+    <parent link="virtual_yaw_link"/>
     <child link="end_effector_link"/>
   </joint>

Commit message: cleanup starter branch

File: bme_ros2_simple_arm/urdf/mogi_arm.xacro (robot description, xacro)
@@ -1,8 +1,4 @@
 <?xml version="1.0"?>
 <robot name="mogi_arm" xmlns:xacro="http://www.ros.org/wiki/xacro">
-  <!-- STEP 3 - RViz colors -->
-  <xacro:include filename="$(find bme_ros2_simple_arm)/urdf/materials.xacro" />
-  <!-- STEP 8 - Gazebo plugin -->
-  <xacro:include filename="$(find bme_ros2_simple_arm)/urdf/mogi_arm.gazebo" />
   <!-- STEP 1 - Global reference link -->
   <link name="world"/>
@@ -35,484 +31,3 @@
     </visual>
   </link>
-  <!-- STEP 4 - Shoulder -->
-  <joint name="shoulder_pan_joint" type="revolute">
-    <limit lower="-3.14" upper="3.14" effort="330.0" velocity="3.14"/>
-    <parent link="base_link"/>
-    <child link="shoulder_link"/>
-    <axis xyz="0 0 1"/>
-    <origin xyz="0.0 0.0 0.05" rpy="0.0 0.0 0.0"/>
-    <dynamics damping="0.0" friction="0.0"/>
-  </joint>
-  <!-- Shoulder link -->
-  <link name="shoulder_link">
-    <inertial>
-      <mass value="0.5"/>
-      <origin xyz="0.0 0.0 0.0" rpy="0.0 0.0 0.0"/>
-      <inertia ixx="0.0014" ixy="0.0" ixz="0.0"
-               iyy="0.0014" iyz="0.0"
-               izz="0.0025"
-      />
-    </inertial>
-    <collision>
-      <geometry>
-        <cylinder radius="0.1" length="0.05"/>
-      </geometry>
-      <origin xyz="0.0 0.0 0.0" rpy="0.0 0.0 0.0"/>
-    </collision>
-    <visual>
-      <geometry>
-        <!-- <cylinder radius="0.1" length="0.05"/> -->
-        <mesh filename = "package://bme_ros2_simple_arm/meshes/shoulder.dae"/>
-      </geometry>
-      <material name="orange"/>
-      <origin xyz="0.0 0.0 0.0" rpy="0.0 0.0 0.0"/>
-    </visual>
-  </link>
-  <!-- Shoulder lift joint -->
-  <joint name="shoulder_lift_joint" type="revolute">
-    <limit lower="-1.5708" upper="1.5708" effort="330.0" velocity="3.14"/>
-    <parent link="shoulder_link"/>
-    <child link="upper_arm_link"/>
-    <axis xyz="0 1 0"/>
-    <origin xyz="0.0 0.0 0.025" rpy="0.0 0.0 0.0"/>
-    <dynamics damping="0.0" friction="0.0"/>
-  </joint>
-  <!-- Upper arm link -->
-  <link name="upper_arm_link">
-    <inertial>
-      <mass value="0.3"/>
-      <origin xyz="0.0 0.0 0.1" rpy="0.0 0.0 0.0"/>
-      <inertia ixx="0.0012" ixy="0.0" ixz="0.0"
-               iyy="0.0012" iyz="0.0"
-               izz="0.0004"
-      />
-    </inertial>
-    <collision>
-      <geometry>
-        <cylinder radius="0.05" length="0.2"/>
-      </geometry>
-      <origin xyz="0.0 0.0 0.1" rpy="0.0 0.0 0.0"/>
-    </collision>
-    <visual>
-      <geometry>
-        <!-- <cylinder radius="0.05" length="0.2"/> -->
-        <mesh filename = "package://bme_ros2_simple_arm/meshes/upper_arm.dae"/>
-      </geometry>
-      <material name="orange"/>
-      <origin xyz="0.0 0.0 0.1" rpy="0.0 0.0 0.0"/>
-    </visual>
-  </link>
-  <!-- STEP 5 - Elbow -->
-  <joint name="elbow_joint" type="revolute">
-    <limit lower="-2.3562" upper="2.3562" effort="150.0" velocity="3.14"/>
-    <parent link="upper_arm_link"/>
-    <child link="forearm_link"/>
-    <axis xyz="0 1 0"/>
-    <origin xyz="0.0 0.0 0.2" rpy="0.0 0.0 0.0"/>
-    <dynamics damping="0.0" friction="0.0"/>
-  </joint>
-  <!-- Forearm link -->
-  <link name="forearm_link">
-    <inertial>
-      <mass value="0.2"/>
-      <origin xyz="0.0 0.0 0.125" rpy="0.0 0.0 0.0"/>
-      <inertia ixx="0.0011" ixy="0.0" ixz="0.0"
-               iyy="0.0011" iyz="0.0"
-               izz="0.0004"
-      />
-    </inertial>
-    <collision>
-      <geometry>
-        <cylinder radius="0.025" length="0.25"/>
-      </geometry>
-      <origin xyz="0.0 0.0 0.125" rpy="0.0 0.0 0.0"/>
-    </collision>
-    <visual>
-      <geometry>
-        <!-- <cylinder radius="0.025" length="0.25"/> -->
-        <mesh filename = "package://bme_ros2_simple_arm/meshes/forearm.dae"/>
-      </geometry>
-      <material name="orange"/>
-      <origin xyz="0.0 0.0 0.125" rpy="0.0 0.0 0.0"/>
-    </visual>
-  </link>
-  <!-- STEP 6 - Wrist -->
-  <joint name="wrist_joint" type="revolute">
-    <limit lower="-2.3562" upper="2.3562" effort="54.0" velocity="3.14"/>
-    <parent link="forearm_link"/>
-    <child link="wrist_link"/>
-    <axis xyz="0 1 0"/>
-    <origin xyz="0.0 0.0 0.25" rpy="0.0 0.0 0.0"/>
-    <dynamics damping="0.0" friction="0.0"/>
-  </joint>
-  <!-- Wrist link -->
-  <link name="wrist_link">
-    <inertial>
-      <mass value="0.1"/>
-      <origin xyz="0.0 0.0 0.05" rpy="0.0 0.0 0.0"/>
-      <inertia ixx="0.00009" ixy="0.0" ixz="0.0"
-               iyy="0.00009" iyz="0.0"
-               izz="0.00002"
-      />
-    </inertial>
-    <collision>
-      <geometry>
-        <cylinder radius="0.02" length="0.1"/>
-      </geometry>
-      <origin xyz="0.0 0.0 0.05" rpy="0.0 0.0 0.0"/>
-    </collision>
-    <visual>
-      <geometry>
-        <!-- <cylinder radius="0.02" length="0.1"/> -->
-        <mesh filename = "package://bme_ros2_simple_arm/meshes/wrist.dae"/>
-      </geometry>
-      <material name="orange"/>
-      <origin xyz="0.0 0.0 0.05" rpy="0.0 0.0 0.0"/>
-    </visual>
-  </link>
-  <!-- STEP 7 - Gripper -->
-  <joint name="gripper_base_joint" type="fixed">
-    <parent link="wrist_link"/>
-    <child link="gripper_base"/>
-    <origin xyz="0.0 0 0.105" rpy="0.0 0 0"/>
-  </joint>
-  <!-- Gripper base link -->
-  <link name="gripper_base">
-    <inertial>
-      <mass value="0.1"/>
-      <origin xyz="0.0 0.0 0.0" rpy="0.0 0.0 0.0"/>
-      <inertia ixx="0.00009" ixy="0.0" ixz="0.0"
-               iyy="0.00009" iyz="0.0"
-               izz="0.00002"
-      />
-    </inertial>
-    <collision>
-      <geometry>
-        <box size=".05 .1 .01"/>
-      </geometry>
-      <origin xyz="0.0 0.0 0.0" rpy="0.0 0.0 0.0"/>
-    </collision>
-    <visual>
-      <geometry>
-        <box size=".05 .1 .01"/>
-      </geometry>
-      <material name="grey"/>
-      <origin xyz="0.0 0.0 0.0" rpy="0.0 0.0 0.0"/>
-    </visual>
-  </link>
-  <!-- Left finger joint -->
-  <joint name="left_finger_joint" type="prismatic">
-    <limit lower="0" upper="0.04" effort="100.0" velocity="4.0"/>
-    <parent link="gripper_base"/>
-    <child link="left_finger"/>
-    <axis xyz="0 1 0"/>
-    <origin xyz="0.0 0.01 0.045" />
-  </joint>
-  <!-- Left finger link -->
-  <link name="left_finger">
-    <inertial>
-      <mass value="0.1"/>
-      <origin xyz="0.0 0.0 0.0" rpy="0.0 0.0 0.0"/>
-      <inertia ixx="0.00009" ixy="0.0" ixz="0.0"
-               iyy="0.00009" iyz="0.0"
-               izz="0.00002"
-      />
-    </inertial>
-    <collision>
-      <geometry>
-        <box size=".04 .01 .08"/>
-      </geometry>
-      <origin xyz="0.0 0.0 0.0" rpy="0.0 0.0 0.0"/>
-    </collision>
-    <visual>
-      <geometry>
-        <box size=".04 .01 .08"/>
-      </geometry>
-      <material name="blue"/>
-      <origin xyz="0.0 0.0 0.0" rpy="0.0 0.0 0.0"/>
-    </visual>
-  </link>
-  <gazebo reference="left_finger">
-    <kp>1000000.0</kp>
-    <kd>100.0</kd>
-    <mu1>15</mu1>
-    <mu2>15</mu2>
-    <fdir1>1 0 0</fdir1>
-    <maxVel>1.0</maxVel>
-    <minDepth>0.002</minDepth>
-  </gazebo>
-  <!-- Right finger joint -->
-  <joint name="right_finger_joint" type="prismatic">
-    <limit lower="0" upper="0.04" effort="100.0" velocity="4.0"/>
-    <parent link="gripper_base"/>
-    <child link="right_finger"/>
-    <axis xyz="0 -1 0"/>
-    <origin xyz="0.0 -0.01 0.045" />
-  </joint>
-  <!-- Right finger link -->
-  <link name="right_finger">
-    <inertial>
-      <mass value="0.1"/>
-      <origin xyz="0.0 0.0 0.0" rpy="0.0 0.0 0.0"/>
-      <inertia ixx="0.00009" ixy="0.0" ixz="0.0"
-               iyy="0.00009" iyz="0.0"
-               izz="0.00002"
-      />
-    </inertial>
-    <collision>
-      <geometry>
-        <box size=".04 .01 .08"/>
-      </geometry>
-      <origin xyz="0.0 0.0 0.0" rpy="0.0 0.0 0.0"/>
-    </collision>
-    <visual>
-      <geometry>
-        <box size=".04 .01 .08"/>
-      </geometry>
-      <material name="blue"/>
-      <origin xyz="0.0 0.0 0.0" rpy="0.0 0.0 0.0"/>
-    </visual>
-  </link>
-  <gazebo reference="right_finger">
-    <kp>1000000.0</kp>
-    <kd>100.0</kd>
-    <mu1>15</mu1>
-    <mu2>15</mu2>
-    <fdir1>1 0 0</fdir1>
-    <maxVel>1.0</maxVel>
-    <minDepth>0.002</minDepth>
-  </gazebo>
-  <!-- STEP 13 - Virtual roll joint -->
-  <joint name="virtual_roll_joint" type="revolute">
-    <limit lower="-3.1415" upper="3.1415" effort="54.0" velocity="3.14"/>
-    <parent link="wrist_link"/>
-    <child link="virtual_roll_link"/>
-    <axis xyz="0 0 1"/>
-    <origin xyz="0.0 0.0 0.175" rpy="0 0 0"/>
-    <dynamics damping="0.0" friction="0.0"/>
-  </joint>
-  <!-- Virtual roll link -->
-  <link name="virtual_roll_link">
-    <visual>
-      <origin xyz="0 0 0" rpy="0 0 0"/>
-      <geometry>
-        <box size="0.01 0.01 0.01" />
-      </geometry>
-      <material name="red"/>
-     </visual>
-    <inertial>
-      <origin xyz="0 0 0" />
-      <mass value="1.0e-03" />
-      <inertia ixx="1.0e-03" ixy="0.0" ixz="0.0"
-               iyy="1.0e-03" iyz="0.0"
-               izz="1.0e-03" />
-    </inertial>
-  </link>
-  <!-- Virtual yaw joint -->
-  <joint name="virtual_yaw_joint" type="revolute">
-    <limit lower="-3.1415" upper="3.1415" effort="54.0" velocity="3.14"/>
-    <parent link="virtual_roll_link"/>
-    <child link="virtual_yaw_link"/>
-    <axis xyz="1 0 0"/>
-    <origin xyz="0.0 0.0 0.0" rpy="0 0 0"/>
-    <dynamics damping="0.0" friction="0.0"/>
-  </joint>
-  <!-- Virtual yaw link -->
-  <link name="virtual_yaw_link">
-    <visual>
-      <origin xyz="0 0 0" rpy="0 0 0"/>
-      <geometry>
-        <box size="0.01 0.01 0.01" />
-      </geometry>
-      <material name="red"/>
-     </visual>
-    <inertial>
-      <origin xyz="0 0 0" />
-      <mass value="1.0e-03" />
-      <inertia ixx="1.0e-03" ixy="0.0" ixz="0.0"
-               iyy="1.0e-03" iyz="0.0"
-               izz="1.0e-03" />
-    </inertial>
-  </link>
-  <!-- STEP 9 - ROS2 control -->
-  <ros2_control name="GazeboSystem" type="system">
-    <hardware>
-      <plugin>gz_ros2_control/GazeboSimSystem</plugin>
-    </hardware>
-    <joint name="shoulder_pan_joint">
-      <command_interface name="position">
-        <param name="min">-2</param>
-        <param name="max">2</param>
-      </command_interface>
-      <state_interface name="position">
-        <param name="initial_value">0.0</param>
-      </state_interface>
-      <state_interface name="velocity"/>
-      <state_interface name="effort"/>
-    </joint>
-    <joint name="shoulder_lift_joint">
-      <command_interface name="position">
-        <param name="min">-2</param>
-        <param name="max">2</param>
-      </command_interface>
-      <state_interface name="position">
-        <param name="initial_value">0.0</param>
-      </state_interface>
-      <state_interface name="velocity"/>
-      <state_interface name="effort"/>
-    </joint>
-    <joint name="elbow_joint">
-      <command_interface name="position">
-        <param name="min">-2</param>
-        <param name="max">2</param>
-      </command_interface>
-      <state_interface name="position">
-        <param name="initial_value">0.0</param>
-      </state_interface>
-      <state_interface name="velocity"/>
-      <state_interface name="effort"/>
-    </joint>
-    <joint name="wrist_joint">
-      <command_interface name="position">
-        <param name="min">-2</param>
-        <param name="max">2</param>
-      </command_interface>
-      <state_interface name="position">
-        <param name="initial_value">0.0</param>
-      </state_interface>
-      <state_interface name="velocity"/>
-      <state_interface name="effort"/>
-    </joint>
-    <joint name="virtual_roll_joint">
-      <command_interface name="position">
-        <param name="min">-2</param>
-        <param name="max">2</param>
-      </command_interface>
-      <state_interface name="position">
-        <param name="initial_value">0.0</param>
-      </state_interface>
-      <state_interface name="velocity"/>
-      <state_interface name="effort"/>
-    </joint>
-    <joint name="virtual_yaw_joint">
-      <command_interface name="position">
-        <param name="min">-2</param>
-        <param name="max">2</param>
-      </command_interface>
-      <state_interface name="position">
-        <param name="initial_value">0.0</param>
-      </state_interface>
-      <state_interface name="velocity"/>
-      <state_interface name="effort"/>
-    </joint>
-    <joint name="left_finger_joint">
-      <command_interface name="position">
-        <param name="min">-2</param>
-        <param name="max">2</param>
-      </command_interface>
-      <state_interface name="position">
-        <param name="initial_value">0.0</param>
-      </state_interface>
-      <state_interface name="velocity"/>
-      <state_interface name="effort"/>
-    </joint>
-    <joint name="right_finger_joint">
-      <command_interface name="position">
-        <param name="min">-2</param>
-        <param name="max">2</param>
-      </command_interface>
-      <state_interface name="position">
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
Commit message: fix end effector position

File: bme_ros2_simple_arm/urdf/mogi_arm.xacro (robot description, xacro)
@@ -431,5 +431,5 @@
   <!-- STEP 10 - End effector -->
   <joint name="end_effector_joint" type="fixed">
-    <origin xyz="0.0 0.0 0.175" rpy="0 0 0"/>
+    <origin xyz="0.0 0.0 0.0" rpy="0 0 0"/>
     <parent link="virtual_yaw_link"/>
     <child link="end_effector_link"/>
